File: autonomous_rc_pcb.kicad_pcb (KiCad board)
At the start: 6 copper layers, 36.5 x 28 mm, 220 parts, among them J9 Micro_SD_Card, P1 USB_A_Vertical, P2 HDMI_PAUL, P3 SMA_SMD, P4 SMA_SMD, P5 SMA_SMD, P7 USB_A_Vertical, U1 MCP1603L, U10 ECMF04-4HSM10, U11 CM1624, U12 ECMF04-4HSM10, U13 USB2514Bi, U14 LAN9514/LAN9514i, U15 Wurth_Magnetics_749010012A, U2 MCP16311/2, U3 MCP16311/2, U4 Autopilot_module, U5 ESD-8040, U6 CC2520, U7 CC2592, U8 CC112X, U9 UBLOX_NEO_M8P, X1 32Mhz, X2 32MHZ, X3 XRCGB24M000F2P00R0, X4 XRCGB25M000F2P00R0

Commit message: beta
beta pcb version 0.001V
Parts:
- added C105: 22uF, Capacitors_SMD:C_0805_HandSoldering, F.Cu at (118.9, 48.4)
- added C106: 22uF, Capacitors_SMD:C_0805_HandSoldering, F.Cu at (118.9, 50.7)
- added D8: 1N5822, PAUL-DIODE-SMD:D_DO-201AD_P5.08mm_Vertical_AnodeUp, F.Cu at (98.7, 45.9)
- added G***: LOGO, Don-UAV_C-Logo:LOGO_DAS, B.Cu at (115.1, 50.4)
- added L29: 4.7uH, Inductors_SMD:L_Taiyo-Yuden_NR-50xx_HandSoldering, F.Cu at (120.1, 43.1)
- added R44: 10k, Resistor_SMD:R_0402_1005Metric, F.Cu at (114.0, 50.7)
- added REF**: MountingHole_3.2mm_M3, Don-Mechanical:MountingHole_3.2mm_M3_Pad_Via, F.Cu at (156.2, 167.3)
- added REF**: MountingHole_3.2mm_M3, Don-Mechanical:MountingHole_3.2mm_M3_Pad_Via, F.Cu at (73.1, 167.4)
- added REF**: MountingHole_3.2mm_M3, Don-Mechanical:MountingHole_3.2mm_M3_Pad_Via, F.Cu at (73.1, 32.0)
- added REF**: MountingHole_3.2mm_M3, Don-Mechanical:MountingHole_3.2mm_M3_Pad_Via, F.Cu at (156.2, 32.0)
- added U16: AP3512E, Package_SO:PowerIntegrations_SO-8, F.Cu at (114.6, 43.0)
- C1: value 10uF50V -> 10nF
- C10: footprint Capacitors_SMD:C_0402 -> Capacitors_SMD:C_0805_HandSoldering
- C11, C2: value 10uF50V -> 10uF
- C12: value 10uF50V -> 10uF; footprint Capacitors_SMD:C_0402 -> Capacitors_SMD:C_0805_HandSoldering
- C14: value 10uF -> 3.3nF
- C5: value 1uF -> 100uF; footprint Capacitors_SMD:C_0402 -> Capacitor_THT:CP_Radial_D8.0mm_P3.50mm
- C7: value 100nF -> 1000uF; footprint Capacitors_SMD:C_0402 -> Capacitor_THT:CP_Radial_D8.0mm_P5.00mm
- L3: value 15uH -> 100uH; footprint Inductors_SMD:L_Abracon_ASPI-3012S -> Inductors_SMD:L_Vishay_IHLP-4040
- R3: value 31.6k -> 26.1k; footprint Resistors_SMD:R_0402 -> Resistor_SMD:R_0402_1005Metric
- R4: footprint Resistors_SMD:R_0402 -> Resistor_SMD:R_0402_1005Metric
- U3: value MCP16311/2 -> LM2576S-12/NOPB; footprint Housings_SSOP:MSOP-8-1EP_3x3mm_Pitch0.65mm -> Package_TO_SOT_SMD:TO-263-5_TabPin3
- moved C11 170.0 mm to (117.5, 35.9)
- moved C6 169.6 mm to (124.9, 31.9)
- moved C13 169.6 mm to (131.1, 29.3)
- moved C2 169.6 mm to (118.8, 35.9)
- moved C4 169.6 mm to (118.5, 33.9)
- moved C9 169.6 mm to (129.8, 29.4)
- moved L2 169.6 mm to (129.0, 33.4)
- moved U2 169.6 mm to (122.7, 34.4)
- moved R1 167.2 mm to (122.5, 31.8)
- moved R2 167.2 mm to (120.4, 31.8)
- moved C1 166.1 mm to (118.5, 38.8), turned to 0 degrees
- moved C12 159.5 mm to (109.3, 42.2), turned to 180 degrees
- moved R4 157.4 mm to (110.6, 46.7)
- moved R3 154.9 mm to (110.6, 44.8), turned to 0 degrees
- moved C14 153.7 mm to (114.0, 48.5)
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Connections:
- C1 pad 1: +28V -> Net-(C1-Pad1)
- C1 pad 2: GND -> Net-(C1-Pad2)
- C10 pad 1: +3V3 -> +12V
- C11 pad 1: +28V -> +12V
- C12 pad 1: +28V -> +12V
- C14 pad 1: +3V3 -> Net-(C14-Pad1)
- C14 pad 2: GND -> Net-(C14-Pad2)
- C2 pad 1: +28V -> +12V
- C5 pad 1: Net-(C5-Pad1) -> +36V
- C7 pad 1: Net-(C7-Pad1) -> +12V
- C7 pad 2: Net-(C7-Pad2) -> GND
- ETHERNET1 pad 6: +12C -> +12V
- L3 pad 1: Net-(C7-Pad2) -> Net-(D8-PadK)
- L3 pad 2: +3V3 -> +12V
- POWER1 pad 1: +28V -> +36V
- R22 pad 1: +28V -> +36V
- U2 pad 3: +28V -> +12V
- U2 pad 4: +28V -> +12V
- U3 pad 1: Net-(R3-Pad2) -> +36V
- U3 pad 2: Net-(C5-Pad1) -> Net-(D8-PadK)
- U3 pad 3: +28V -> GND
- U3 pad 4: +28V -> +12V
Routing:
- net +5V: track 327.5 -> 445.7 mm, vias 0 -> 4
- net /VBAT_ADC: track 0.00 -> 117.1 mm, vias 0 -> 2
- net +12V: track 0.00 -> 71.6 mm, vias 0 -> 1
- net GND: track 290.9 -> 361.3 mm, vias 265 -> 299
- net +36V: track 0.00 -> 26.3 mm
- net Net-(D8-PadK): track 0.00 -> 26.1 mm
- net +3V3: track 108.4 -> 126.1 mm, vias 44 -> 51
- net /UBLOX/RTK_STAT: track 92.1 -> 108.7 mm, vias 0 -> 2
- net Net-(C1-Pad2): track 0.00 -> 16.5 mm
- net Net-(C30-Pad1): track 0.00 -> 13.1 mm
- net Net-(L17-Pad2): track 4.70 -> 12.6 mm
- net Net-(L18-Pad2): track 26.9 -> 34.4 mm
- net Net-(C6-Pad2): track 0.00 -> 5.53 mm
- net /das_board/PA1_PWM: track 45.8 -> 49.8 mm
- net /das_board/PB9_PWM: track 74.1 -> 70.3 mm
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- added copper zone on B.Cu, net GND
- added copper zone on F.Cu, net GND
- added copper zone on In1.Cu, net GND
- added copper zone on In2.Cu, net GND
Other:
- board size 36.5 x 28 mm -> 91.1 x 143.4 mm

Commit message: added rf stitching, connector names
Parts:
- 1V8: renamed from D5; value 3V3 -> (none)
- renumbered P3 to 2.4GHz, D6 to 3V3, P4 to 420-470MHz, D7 to 5V, P5 to RTK, D1 to RTK_STAT, U9 to UBLOX_NEO_M8P
Routing:
- net /das_board/PA1_PWM: track 49.8 -> 53.6 mm
- net GND: track 361.3 -> 364.4 mm
- net (no net): vias 0 -> 101
