File: CC1120.sch (KiCad schematic (older format))
At the start: 39 parts, among them P4 SMA_SMD, U8 CC112X, X2 32MHZ

Commit message: tuned rf
added u.fl connectors to tune line 
moved some lines under rf components
Parts:
- renumbered P4 to 420-470MHz1
Changed lines of the file:
@@
 $Descr A4 11693 8268
 encoding utf-8
-Sheet 5 10
+Sheet 4 10
 Title "CC1120 420 - 470 MHz"
 Date "2016-02-11"
@@
 $EndComp
 $Comp
-L GND #PWR0103
+L GND #PWR0104
 U 1 1 5AEB2B37
 P 1550 3700
-F 0 "#PWR0103" H 1550 3450 50  0001 C CNN
+F 0 "#PWR0104" H 1550 3450 50  0001 C CNN
 F 1 "GND" H 1550 3550 50  0000 C CNN
 F 2 "" H 1550 3700 50  0001 C CNN
@@
 $EndComp
 $Comp
-L GND #PWR0104
+L GND #PWR0105
 U 1 1 5AEB2BC1
 P 1050 2850
-F 0 "#PWR0104" H 1050 2600 50  0001 C CNN
+F 0 "#PWR0105" H 1050 2600 50  0001 C CNN
 F 1 "GND" H 1050 2700 50  0000 C CNN
 F 2 "" H 1050 2850 50  0001 C CNN
@@
 $EndComp
 $Comp
-L GND #PWR0105
+L GND #PWR0106
 U 1 1 5AEB301E
 P 1050 3250
-F 0 "#PWR0105" H 1050 3000 50  0001 C CNN
+F 0 "#PWR0106" H 1050 3000 50  0001 C CNN
 F 1 "GND" H 1050 3100 50  0000 C CNN
 F 2 "" H 1050 3250 50  0001 C CNN
@@
 $EndComp
 $Comp
-L GND #PWR0106
+L GND #PWR0107
 U 1 1 5AEB34C4
 P 3100 5000
-F 0 "#PWR0106" H 3100 4750 50  0001 C CNN
+F 0 "#PWR0107" H 3100 4750 50  0001 C CNN
 F 1 "GND" H 3100 4850 50  0000 C CNN
 F 2 "" H 3100 5000 50  0001 C CNN
@@
 VDD_REG
 $Comp
-L GND #PWR0107
+L GND #PWR0108
 U 1 1 5AEB3A51
 P 3450 4850
-F 0 "#PWR0107" H 3450 4600 50  0001 C CNN
+F 0 "#PWR0108" H 3450 4600 50  0001 C CNN
 F 1 "GND" H 3450 4700 50  0000 C CNN
 F 2 "" H 3450 4850 50  0001 C CNN
@@
 $EndComp
 $Comp
-L GND #PWR0108
+L GND #PWR0109
 U 1 1 5AEB3B15
 P 3800 4800
-F 0 "#PWR0108" H 3800 4550 50  0001 C CNN
+F 0 "#PWR0109" H 3800 4550 50  0001 C CNN
 F 1 "GND" H 3800 4650 50  0000 C CNN
 F 2 "" H 3800 4800 50  0001 C CNN
@@
 $EndComp
 $Comp
-L GND #PWR0109
+L GND #PWR0110
 U 1 1 5AEB3B8E
 P 4050 4750
-F 0 "#PWR0109" H 4050 4500 50  0001 C CNN
+F 0 "#PWR0110" H 4050 4500 50  0001 C CNN
 F 1 "GND" H 4050 4600 50  0000 C CNN
 F 2 "" H 4050 4750 50  0001 C CNN
@@
 $EndComp
 $Comp
-L GND #PWR0110
+L GND #PWR0111
 U 1 1 5AF041C2
 P 2550 2050
-F 0 "#PWR0110" H 2550 1800 50  0001 C CNN
+F 0 "#PWR0111" H 2550 1800 50  0001 C CNN
 F 1 "GND" H 2550 1900 50  0000 C CNN
 F 2 "" H 2550 2050 50  0001 C CNN
@@
 VDD_REG
 $Comp
-L GND #PWR0111
+L GND #PWR0112
 U 1 1 5AF0476E
 P 4350 1450
-F 0 "#PWR0111" H 4350 1200 50  0001 C CNN
+F 0 "#PWR0112" H 4350 1200 50  0001 C CNN
 F 1 "GND" H 4350 1300 50  0000 C CNN
 F 2 "" H 4350 1450 50  0001 C CNN
@@
 $EndComp
 $Comp
-L GND #PWR0112
+L GND #PWR0113
 U 1 1 5AF06432
 P 2300 1700
-F 0 "#PWR0112" H 2300 1450 50  0001 C CNN
+F 0 "#PWR0113" H 2300 1450 50  0001 C CNN
 F 1 "GND" H 2300 1550 50  0000 C CNN
 F 2 "" H 2300 1700 50  0001 C CNN
@@
 $EndComp
 $Comp
-L GND #PWR0113
+L GND #PWR0114
 U 1 1 5AF069C0
 P 1450 2000
-F 0 "#PWR0113" H 1450 1750 50  0001 C CNN
+F 0 "#PWR0114" H 1450 1750 50  0001 C CNN
 F 1 "GND" H 1450 1850 50  0000 C CNN
 F 2 "" H 1450 2000 50  0001 C CNN
@@
 $EndComp
 $Comp
-L GND #PWR0114
+L GND #PWR0115
 U 1 1 5AF071F6
 P 4600 2700
-F 0 "#PWR0114" H 4600 2450 50  0001 C CNN
+F 0 "#PWR0115" H 4600 2450 50  0001 C CNN
 F 1 "GND" H 4600 2550 50  0000 C CNN
 F 2 "" H 4600 2700 50  0001 C CNN
@@
 $EndComp
 $Comp
-L GND #PWR0115
+L GND #PWR0116
 U 1 1 5AF0776A
 P 4950 2700
-F 0 "#PWR0115" H 4950 2450 50  0001 C CNN
+F 0 "#PWR0116" H 4950 2450 50  0001 C CNN
 F 1 "GND" H 4950 2550 50  0000 C CNN
 F 2 "" H 4950 2700 50  0001 C CNN
@@
 $EndComp
 $Comp
-L GND #PWR0116
+L GND #PWR0117
 U 1 1 5AF07DD6
 P 6100 2500
-F 0 "#PWR0116" H 6100 2250 50  0001 C CNN
+F 0 "#PWR0117" H 6100 2250 50  0001 C CNN
 F 1 "GND" H 6100 2350 50  0000 C CNN
 F 2 "" H 6100 2500 50  0001 C CNN
@@
 $EndComp
 $Comp
-L GND #PWR0117
+L GND #PWR0118
 U 1 1 5AF08A03
 P 6550 3900
-F 0 "#PWR0117" H 6550 3650 50  0001 C CNN
+F 0 "#PWR0118" H 6550 3650 50  0001 C CNN
 F 1 "GND" H 6550 3750 50  0000 C CNN
 F 2 "" H 6550 3900 50  0001 C CNN
@@
 	8500 4650 9300 4650
 $Comp
-L GND #PWR0118
+L GND #PWR0119
 U 1 1 5AF0B670
 P 7700 5150
-F 0 "#PWR0118" H 7700 4900 50  0001 C CNN
+F 0 "#PWR0119" H 7700 4900 50  0001 C CNN
 F 1 "GND" H 7700 5000 50  0000 C CNN
 F 2 "" H 7700 5150 50  0001 C CNN
@@
 	5700 5600 5700 5700
 $Comp
-L GND #PWR0119
+L GND #PWR0120
 U 1 1 5AF0C06A
 P 5400 6650
-F 0 "#PWR0119" H 5400 6400 50  0001 C CNN
+F 0 "#PWR0120" H 5400 6400 50  0001 C CNN
 F 1 "GND" H 5400 6500 50  0000 C CNN
 F 2 "" H 5400 6650 50  0001 C CNN
@@
 $EndComp
 $Comp
-L GND #PWR0120
+L GND #PWR0121
 U 1 1 5AF0C0CA
 P 5700 6650
-F 0 "#PWR0120" H 5700 6400 50  0001 C CNN
+F 0 "#PWR0121" H 5700 6400 50  0001 C CNN
 F 1 "GND" H 5700 6500 50  0000 C CNN
 F 2 "" H 5700 6650 50  0001 C CNN
@@
 	5400 6600 5400 6650
 $Comp
-L GND #PWR0121
+L GND #PWR0122
 U 1 1 5AF0D20D
 P 9900 5150
-F 0 "#PWR0121" H 9900 4900 50  0001 C CNN
+F 0 "#PWR0122" H 9900 4900 50  0001 C CNN
 F 1 "GND" H 9900 5000 50  0000 C CNN
 F 2 "" H 9900 5150 50  0001 C CNN
@@
 $EndComp
 $Comp
-L SMA_SMD P4
+L SMA_SMD 420-470MHz1
 U 1 1 5AF0DE95
 P 9550 4650
-F 0 "P4" H 9500 5100 60  0000 C CNN
+F 0 "420-470MHz1" H 9500 5100 60  0000 C CNN
 F 1 "SMA_SMD" H 9650 5000 60  0000 C CNN
 F 2 "Connectors:SMA_THT_Jack_Straight" H 9650 5200 60  0001 C CNN
@@
 VDD_REG
 $Comp
-L +5V #PWR0122
+L +5V #PWR0123
 U 1 1 5AF23DB6
 P 6800 1500
-F 0 "#PWR0122" H 6800 1350 50  0001 C CNN
+F 0 "#PWR0123" H 6800 1350 50  0001 C CNN
 F 1 "+5V" H 6800 1640 50  0000 C CNN
 F 2 "" H 6800 1500 50  0001 C CNN
