File: UBLOX.sch (KiCad schematic (older format))
At the start: 6 parts, among them P5 SMA_SMD, U9 UBLOX_NEO_M8P

Commit message: tuned rf
added u.fl connectors to tune line 
moved some lines under rf components
Parts:
- renumbered P5 to RTK1
Changed lines of the file:
@@
 $Descr A4 11693 8268
 encoding utf-8
-Sheet 6 10
+Sheet 5 10
 Title ""
 Date ""
@@
 Connection ~ 4750 4250
 $Comp
-L GND #PWR0123
+L GND #PWR0124
 U 1 1 5AF25ABC
 P 4750 4600
-F 0 "#PWR0123" H 4750 4350 50  0001 C CNN
+F 0 "#PWR0124" H 4750 4350 50  0001 C CNN
 F 1 "GND" H 4750 4450 50  0000 C CNN
 F 2 "" H 4750 4600 50  0001 C CNN
@@
 Connection ~ 4550 3950
 $Comp
-L GND #PWR0124
+L GND #PWR0125
 U 1 1 5AF25B89
 P 4550 4600
-F 0 "#PWR0124" H 4550 4350 50  0001 C CNN
+F 0 "#PWR0125" H 4550 4350 50  0001 C CNN
 F 1 "GND" H 4550 4450 50  0000 C CNN
 F 2 "" H 4550 4600 50  0001 C CNN
@@
 $EndComp
 $Comp
-L SMA_SMD P5
+L SMA_SMD RTK1
 U 1 1 5AF25C93
 P 7200 2850
-F 0 "P5" H 7150 3300 60  0000 C CNN
+F 0 "RTK1" H 7150 3300 60  0000 C CNN
 F 1 "SMA_SMD" H 7300 3200 60  0000 C CNN
 F 2 "Connectors:SMA_THT_Jack_Straight" H 7300 3400 60  0001 C CNN
@@
 	8250 3500 8250 3650
 $Comp
-L GND #PWR0125
+L GND #PWR0126
 U 1 1 5AF25F3C
 P 8250 4050
-F 0 "#PWR0125" H 8250 3800 50  0001 C CNN
+F 0 "#PWR0126" H 8250 3800 50  0001 C CNN
 F 1 "GND" H 8250 3900 50  0000 C CNN
 F 2 "" H 8250 4050 50  0001 C CNN
@@
 Connection ~ 7700 2700
 $Comp
-L GND #PWR0126
+L GND #PWR0127
 U 1 1 5AF26136
 P 7700 3050
-F 0 "#PWR0126" H 7700 2800 50  0001 C CNN
+F 0 "#PWR0127" H 7700 2800 50  0001 C CNN
 F 1 "GND" H 7700 2900 50  0000 C CNN
 F 2 "" H 7700 3050 50  0001 C CNN
@@
 Connection ~ 7200 3500
 $Comp
-L +3V3 #PWR0127
+L +3V3 #PWR0128
 U 1 1 5AF26291
 P 4550 3100
-F 0 "#PWR0127" H 4550 2950 50  0001 C CNN
+F 0 "#PWR0128" H 4550 2950 50  0001 C CNN
 F 1 "+3V3" H 4550 3240 50  0000 C CNN
 F 2 "" H 4550 3100 50  0001 C CNN
