File: USB_HOST.sch (KiCad schematic (older format))
At the start: 20 parts, among them U13 USB2514Bi, X3 XRCGB24M000F2P00R0

Commit message: tuned rf
added u.fl connectors to tune line 
moved some lines under rf components
Parts:
- C64, C67: footprint Capacitors_SMD:C_0402 -> Capacitor_SMD:C_0603_1608Metric
Changed lines of the file:
@@
 $EndDescr
 $Comp
-L +3V3 #PWR0212
+L +3V3 #PWR0213
 U 1 1 5AF435FB
 P 3200 2000
-F 0 "#PWR0212" H 3200 1850 50  0001 C CNN
+F 0 "#PWR0213" H 3200 1850 50  0001 C CNN
 F 1 "+3V3" H 3200 2140 50  0000 C CNN
 F 2 "" H 3200 2000 60  0000 C CNN
@@
 $EndComp
 $Comp
-L GND #PWR0213
+L GND #PWR0214
 U 1 1 5AF435FD
 P 7500 5400
-F 0 "#PWR0213" H 7500 5150 50  0001 C CNN
+F 0 "#PWR0214" H 7500 5150 50  0001 C CNN
 F 1 "GND" H 7500 5250 50  0000 C CNN
 F 2 "" H 7500 5400 60  0000 C CNN
@@
 $EndComp
 $Comp
-L GND #PWR0214
+L GND #PWR0215
 U 1 1 5AF43600
 P 4450 4050
-F 0 "#PWR0214" H 4450 3800 50  0001 C CNN
+F 0 "#PWR0215" H 4450 3800 50  0001 C CNN
 F 1 "GND" H 4450 3900 50  0000 C CNN
 F 2 "" H 4450 4050 60  0000 C CNN
@@
 $EndComp
 $Comp
-L GND #PWR0215
+L GND #PWR0216
 U 1 1 5AF43602
 P 7200 5400
-F 0 "#PWR0215" H 7200 5150 50  0001 C CNN
+F 0 "#PWR0216" H 7200 5150 50  0001 C CNN
 F 1 "GND" H 7200 5250 50  0000 C CNN
 F 2 "" H 7200 5400 60  0000 C CNN
@@
 $EndComp
 $Comp
-L GND #PWR0216
+L GND #PWR0217
 U 1 1 5AF43604
 P 7850 4800
-F 0 "#PWR0216" H 7850 4550 50  0001 C CNN
+F 0 "#PWR0217" H 7850 4550 50  0001 C CNN
 F 1 "GND" H 7850 4650 50  0000 C CNN
 F 2 "" H 7850 4800 60  0000 C CNN
@@
 $EndComp
 $Comp
-L GND #PWR0217
+L GND #PWR0218
 U 1 1 5AF43606
 P 4250 4650
-F 0 "#PWR0217" H 4250 4400 50  0001 C CNN
+F 0 "#PWR0218" H 4250 4400 50  0001 C CNN
 F 1 "GND" H 4250 4500 50  0000 C CNN
 F 2 "" H 4250 4650 60  0000 C CNN
@@
 F 0 "C67" H 4660 4620 50  0000 L CNN
 F 1 "9p" H 4660 4470 50  0000 L CNN
-F 2 "Capacitors_SMD:C_0402" H 4650 4550 60  0001 C CNN
+F 2 "Capacitor_SMD:C_0603_1608Metric" H 4650 4550 60  0001 C CNN
 F 3 "" H 4650 4550 60  0000 C CNN
 	1    4650 4550
@@
 F 0 "C64" H 4260 4620 50  0000 L CNN
 F 1 "9p" H 4260 4470 50  0000 L CNN
-F 2 "Capacitors_SMD:C_0402" H 4250 4550 60  0001 C CNN
+F 2 "Capacitor_SMD:C_0603_1608Metric" H 4250 4550 60  0001 C CNN
 F 3 "" H 4250 4550 60  0000 C CNN
 F 4 "GRM1555C1H9R0CA01D" H 4250 4550 60  0001 C CNN "MPN"
@@
 $EndComp
 $Comp
-L GND #PWR0218
+L GND #PWR0219
 U 1 1 5AF43610
 P 4700 2400
-F 0 "#PWR0218" H 4700 2150 50  0001 C CNN
+F 0 "#PWR0219" H 4700 2150 50  0001 C CNN
 F 1 "GND" H 4700 2250 50  0000 C CNN
 F 2 "" H 4700 2400 60  0000 C CNN
@@
 $EndComp
 $Comp
-L GND #PWR0219
+L GND #PWR0220
 U 1 1 5AF43611
 P 4450 2400
-F 0 "#PWR0219" H 4450 2150 50  0001 C CNN
+F 0 "#PWR0220" H 4450 2150 50  0001 C CNN
 F 1 "GND" H 4450 2250 50  0000 C CNN
 F 2 "" H 4450 2400 60  0000 C CNN
@@
 $EndComp
 $Comp
-L GND #PWR0220
+L GND #PWR0221
 U 1 1 5AF43612
 P 4200 2400
-F 0 "#PWR0220" H 4200 2150 50  0001 C CNN
+F 0 "#PWR0221" H 4200 2150 50  0001 C CNN
 F 1 "GND" H 4200 2250 50  0000 C CNN
 F 2 "" H 4200 2400 60  0000 C CNN
@@
 $EndComp
 $Comp
-L GND #PWR0221
+L GND #PWR0222
 U 1 1 5AF43613
 P 3950 2400
-F 0 "#PWR0221" H 3950 2150 50  0001 C CNN
+F 0 "#PWR0222" H 3950 2150 50  0001 C CNN
 F 1 "GND" H 3950 2250 50  0000 C CNN
 F 2 "" H 3950 2400 60  0000 C CNN
@@
 $EndComp
 $Comp
-L GND #PWR0222
+L GND #PWR0223
 U 1 1 5AF43614
 P 3700 2400
-F 0 "#PWR0222" H 3700 2150 50  0001 C CNN
+F 0 "#PWR0223" H 3700 2150 50  0001 C CNN
 F 1 "GND" H 3700 2250 50  0000 C CNN
 F 2 "" H 3700 2400 60  0000 C CNN
@@
 $EndComp
 $Comp
-L GND #PWR0223
+L GND #PWR0224
 U 1 1 5AF43615
 P 3450 2400
-F 0 "#PWR0223" H 3450 2150 50  0001 C CNN
+F 0 "#PWR0224" H 3450 2150 50  0001 C CNN
 F 1 "GND" H 3450 2250 50  0000 C CNN
 F 2 "" H 3450 2400 60  0000 C CNN
@@
 $EndComp
 $Comp
-L GND #PWR0224
+L GND #PWR0225
 U 1 1 5AF43616
 P 3200 2400
-F 0 "#PWR0224" H 3200 2150 50  0001 C CNN
+F 0 "#PWR0225" H 3200 2150 50  0001 C CNN
 F 1 "GND" H 3200 2250 50  0000 C CNN
 F 2 "" H 3200 2400 60  0000 C CNN
@@
 $EndComp
 $Comp
-L GND #PWR0225
+L GND #PWR0226
 U 1 1 5AF43617
 P 4450 4650
-F 0 "#PWR0225" H 4450 4400 50  0001 C CNN
+F 0 "#PWR0226" H 4450 4400 50  0001 C CNN
 F 1 "GND" H 4450 4500 50  0000 C CNN
 F 2 "" H 4450 4650 60  0000 C CNN
@@
 $EndComp
 $Comp
-L GND #PWR0226
+L GND #PWR0227
 U 1 1 5AF43618
 P 4650 4650
-F 0 "#PWR0226" H 4650 4400 50  0001 C CNN
+F 0 "#PWR0227" H 4650 4400 50  0001 C CNN
 F 1 "GND" H 4650 4500 50  0000 C CNN
 F 2 "" H 4650 4650 60  0000 C CNN
@@
 pin 15
 $Comp
-L +3V3 #PWR0227
+L +3V3 #PWR0228
 U 1 1 5AF43619
 P 4450 3300
-F 0 "#PWR0227" H 4450 3150 50  0001 C CNN
+F 0 "#PWR0228" H 4450 3150 50  0001 C CNN
 F 1 "+3V3" H 4450 3440 50  0000 C CNN
 F 2 "" H 4450 3300 60  0000 C CNN
@@
 $EndComp
 $Comp
-L GND #PWR0228
+L GND #PWR0229
 U 1 1 5AF4361A
 P 8650 4400
-F 0 "#PWR0228" H 8650 4150 50  0001 C CNN
+F 0 "#PWR0229" H 8650 4150 50  0001 C CNN
 F 1 "GND" H 8650 4250 50  0000 C CNN
 F 2 "" H 8650 4400 60  0000 C CNN
@@
 $EndComp
 $Comp
-L GND #PWR0229
+L GND #PWR0230
 U 1 1 5AF4361D
 P 8500 4400
-F 0 "#PWR0229" H 8500 4150 50  0001 C CNN
+F 0 "#PWR0230" H 8500 4150 50  0001 C CNN
 F 1 "GND" H 8500 4250 50  0000 C CNN
 F 2 "" H 8500 4400 60  0000 C CNN
@@
 $EndComp
 $Comp
-L GND #PWR0230
+L GND #PWR0231
 U 1 1 5AF4361E
 P 8100 4400
-F 0 "#PWR0230" H 8100 4150 50  0001 C CNN
+F 0 "#PWR0231" H 8100 4150 50  0001 C CNN
 F 1 "GND" H 8100 4250 50  0000 C CNN
 F 2 "" H 8100 4400 60  0000 C CNN
@@
 $EndComp
 $Comp
-L GND #PWR0231
+L GND #PWR0232
 U 1 1 5AF43621
 P 7950 4400
-F 0 "#PWR0231" H 7950 4150 50  0001 C CNN
+F 0 "#PWR0232" H 7950 4150 50  0001 C CNN
 F 1 "GND" H 7950 4250 50  0000 C CNN
 F 2 "" H 7950 4400 60  0000 C CNN
@@
 DN_USB6+
 $Comp
-L GND #PWR0232
+L GND #PWR0233
 U 1 1 5AF43624
 P 5000 5100
-F 0 "#PWR0232" H 5000 4850 50  0001 C CNN
+F 0 "#PWR0233" H 5000 4850 50  0001 C CNN
 F 1 "GND" H 5000 4950 50  0000 C CNN
 F 2 "" H 5000 5100 60  0000 C CNN
@@
 NoConn ~ 5100 4450
 $Comp
-L +3V3 #PWR0233
+L +3V3 #PWR0234
 U 1 1 5AF43643
 P 4900 3550
-F 0 "#PWR0233" H 4900 3400 50  0001 C CNN
+F 0 "#PWR0234" H 4900 3400 50  0001 C CNN
 F 1 "+3V3" H 4900 3690 50  0000 C CNN
 F 2 "" H 4900 3550 60  0000 C CNN
